File: hardware/teensy/xen_teensy_motherboard_8cv_mki.sch (EAGLE design)
At the start: 354 parts, among them IC1 TL074PW, IC10 TEXAS_INSTRUMENTS_DAC8164IBPW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, IC11 TEXAS_INSTRUMENTS_DAC8164IBPW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, IC12 LM4040-10V, IC2 MCP23S17SO, IC3 MCP6004, IC4 MCP6004, IC5 TL074PW, IC6 TEENSY41-OUTER, IC7 R-78E5.0-0.5, IC8 LM4040-5V, IC9 MCP6004, P1 HEADER/MALE/01NOBORDER, P10 HEADER/MALE/01NOBORDER, P11 HEADER/MALE/01NOBORDER, P12 HEADER/MALE/01NOBORDER, P13 HEADER/MALE/01NOBORDER, P14 HEADER/MALE/01NOBORDER, P15 HEADER/MALE/01NOBORDER, P16 HEADER/MALE/01NOBORDER, P17 HEADER/MALE/01NOBORDER, P18 HEADER/MALE/01NOBORDER, P19 HEADER/MALE/01NOBORDER, P2 HEADER/MALE/01NOBORDER, P20 HEADER/MALE/01NOBORDER, P21 HEADER/MALE/01NOBORDER, P22 HEADER/MALE/01NOBORDER, P23 HEADER/MALE/01NOBORDER, P24 HEADER/MALE/01NOBORDER, P25 HEADER/MALE/01NOBORDER, P26 HEADER/MALE/01NOBORDER, P27 HEADER/MALE/01NOBORDER, P28 HEADER/MALE/01NOBORDER, P29 HEADER/MALE/01NOBORDER, P3 HEADER/MALE/01NOBORDER, P30 HEADER/MALE/01NOBORDER, P31 HEADER/MALE/01NOBORDER, P32 HEADER/MALE/01NOBORDER, P33 HEADER/MALE/01NOBORDER, P34 HEADER/MALE/01NOBORDER, P35 HEADER/MALE/01NOBORDER, P36 HEADER/MALE/01NOBORDER, P37 HEADER/MALE/01NOBORDER, P38 HEADER/MALE/01NOBORDER, P39 HEADER/MALE/01NOBORDER, P4 HEADER/MALE/01NOBORDER, P40 HEADER/MALE/01NOBORDER, P41 HEADER/MALE/01NOBORDER, P42 HEADER/MALE/01NOBORDER, P43 HEADER/MALE/01NOBORDER, P44 HEADER/MALE/01NOBORDER, P45 HEADER/MALE/01NOBORDER, P46 HEADER/MALE/01NOBORDER, P47 HEADER/MALE/01NOBORDER, P48 HEADER/MALE/01NOBORDER, P49 HEADER/MALE/01NOBORDER, P5 HEADER/MALE/01NOBORDER, P50 HEADER/MALE/01NOBORDER, P6 HEADER/MALE/01NOBORDER, P7 HEADER/MALE/01NOBORDER, P8 HEADER/MALE/01NOBORDER, P9 HEADER/MALE/01NOBORDER, Q1 BF170, Q10 BF170, Q11 BF170, Q12 BF170, Q13 BF170, Q14 BF170, Q15 BF170, Q16 BF170, Q2 BF170, Q3 BF170, Q4 BF170, Q5 BF170, Q6 BF170, Q7 BF170, Q8 BF170, Q9 BF170

Commit message: Added Wire.h
Parts:
- removed C28, C29, C30, C31: 1nF, capacitors:CAPACITORC0603
- removed C35: 470nF, capacitors:CAPACITORC0603
- removed CV10, CV11, CV12, CV13B, CV14B, CV15B, CV16B, CV9: HEADER/MALE/01, connectors:HEADER/MALE/01
- removed IC12: LM4040-10V, ic_voltage_reg:LM4040CYM3-2.5
- removed IC9: MCP6004, ic_analogue:TL074PW
- removed P20, P43, P48: HEADER/MALE/01NOBORDER, connectors:HEADER/MALE/01NOBORDER
- removed R117: 1K, resistors:RESISTOR
- removed R91, R95: 33k, resistors:RESISTOR
- removed R92, R93, R94, R96, R97, R98: 100k, resistors:RESISTOR
- added OFFSET, PT1, PT2, PT3, PT4, PT5, PT6, PT7, PT8: HEADER/MALE/01, connectors:HEADER/MALE/01
- added U1: 74HC405174HC4051_SO16, ic_analogue:74HC405174HC4051_SO16
- R83, R87: value 33k -> 120k
- R84, R85, R86, R88, R89, R90: value 100k -> 120k
- renumbered CV10B to CV6B, CV11B to CV5B, CV12B to CV8B, CV9B to CV7B
Connections:
- removed net -10VREF: C35.2, IC12.A, R117.1
- removed net N$102: CV9.3, R92.1
- removed net N$103: C30.1, IC9C.-IN, R91.1, R92.2, R93.2, R94.2
- removed net N$75: C28.1, IC9A.-IN, R83.1, R84.2, R85.2, R86.2
- removed net N$76: CV13B.3, R85.1
- removed net N$77: CV11.3, R84.1
- removed net N$78: C29.1, IC9B.-IN, R87.1, R88.2, R89.2, R90.2
- removed net N$79: CV10.3, R89.1
- removed net N$80: CV14B.3, R90.1
- removed net N$81: C31.1, IC9D.-IN, R95.1, R96.2, R97.2, R98.2
- removed net N$82: CV12.3, R96.1
- removed net N$83: CV16B.3, R97.1
- removed net N$84: CV15B.3, R93.1
- new net N$41: PT1.3, U1.Y0
- new net N$52: PT2.3, U1.Y1
- new net N$54: PT3.3, U1.Y2
- new net N$56: PT4.3, U1.Y3
- new net N$59: PT5.3, U1.Y4
- new net N$62: PT6.3, U1.Y5
- new net N$64: PT7.3, U1.Y6
- new net N$66: PT8.3, U1.Y7
- new net OFFSET: OFFSET.3, R83.1, R84.1, R85.1, R86.1, R87.1, R88.1, R89.1, R90.1
- net -12V: no longer R117.2
- net -5VREF: no longer R86.1, R88.1, R94.1, R98.1
- net 3.3V: no longer C32.2, IC9P.V+
- net 5V: now also C32.2, U1.VCC
- net ADC10: now also U1.S1; no longer C31.2, IC9D.OUT, R95.2
- net ADC11: now also U1.S0; no longer C28.2, IC9A.OUT, R83.2
- net ADC8: now also U1.Z; no longer C30.2, IC9C.OUT, R91.2
- net ADC9: now also U1.S2; no longer C29.2, IC9B.OUT, R87.2
- net N$12: now also R86.2
- net N$2: now also R83.2
- net N$20: now also R90.2
- net N$27: now also CV3B.3; no longer CV1B.3
- net N$28: now also R89.2
- net N$34: now also CV1B.3; no longer CV3B.3
- net N$43: now also R88.2
- net N$48: now also R87.2
- net N$5: now also R84.2
- net N$9: now also R85.2
- net PE: now also U1.!E!, U1.GND, U1.VEE; no longer C35.1, IC12.C, IC9A.+IN, IC9B.+IN, IC9C.+IN, IC9D.+IN, IC9P.V-
Other:
- moved on the sheet: C12, C13, C19, C22, C32, C4, C5, C8, C9, CV1B, CV3B, CVO1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

Commit message: Fixed bug setting index to 0
Parts:
- removed U1: 74HC405174HC4051_SO16, ic_analogue:74HC405174HC4051_SO16
- added 3.3VA, 3.3VA1, 3.3VA2, 3.3VA3: HEADER/MALE/01, connectors:HEADER/MALE/01
- added C28, C29: 22uF, capacitors:CAPACITORC0805
- added C30: 10uF, capacitors:CAPACITOR/POLARIZEDSMDB
- added IC12: CD4051CD4051_SO16, ic_analogue:CD4051CD4051_SO16
- added IC9: 3.3V, ic_voltage_reg:LD2981LD2981-SOT89
- added L2: INDUCTORL0603, resistors:INDUCTORL0603
Connections:
- new net 3.3V_A: 3.3VA.3, 3.3VA1.3, 3.3VA2.3, 3.3VA3.3, C15.2, C18.2, C30.+, C32.2, IC10.AVDD, IC11.AVDD, IC12.VCC, IC3P.V+, IC4P.V+, IC9.VOUT
- new net N$72: C29.2, IC9.VIN, L2.2
- net +12V: now also L2.1
- net 3.3V: no longer C15.2, C18.2, IC10.AVDD, IC11.AVDD, IC3P.V+, IC4P.V+
- net 5V: no longer C32.2, U1.VCC
- net ADC10: now also IC12.S1; no longer U1.S1
- net ADC11: now also IC12.S0; no longer U1.S0
- net ADC8: now also IC12.Z; no longer U1.Z
- net ADC9: now also IC12.S2; no longer U1.S2
- net N$41: now also IC12.Y4, PT5.3; no longer PT1.3, U1.Y0
- net N$51: now also C28.2
- net N$52: now also IC12.Y5, PT6.3; no longer PT2.3, U1.Y1
- net N$54: now also IC12.Y3, PT4.3; no longer PT3.3, U1.Y2
- net N$56: now also IC12.Y2, PT3.3; no longer PT4.3, U1.Y3
- net N$59: now also IC12.Y0, PT1.3; no longer PT5.3, U1.Y4
- net N$62: now also IC12.Y1, PT2.3; no longer PT6.3, U1.Y5
- net N$64: now also IC12.Y6; no longer U1.Y6
- net N$66: now also IC12.Y7; no longer U1.Y7
- net PE: now also C28.1, C29.1, C30.-, IC12.!E!, IC12.GND, IC12.VEE, IC9.GND; no longer U1.!E!, U1.GND, U1.VEE
Other:
- moved on the sheet: +V, +V1, +V2, +V3, +V4, +V5, -V, -V1, -V2, -V3, -V4, -V5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

Commit message: Updated hardware
Parts:
- added R91, R92, R93, R94: 0R, resistors:RESISTOR
Connections:
- net ADC10: now also R93.2
- net ADC11: now also R94.2
- net ADC8: now also R91.2
- net ADC9: now also R92.2
- net N$52: now also PT8.3; no longer PT6.3
- net N$54: now also PT1.3, R94.1; no longer PT4.3
- net N$56: now also PT4.3, R91.1; no longer PT3.3
- net N$59: now also PT2.3, R93.1; no longer PT1.3
- net N$62: now also PT3.3, R92.1; no longer PT2.3
- net N$64: now also PT6.3; no longer PT7.3
- net N$66: now also PT7.3; no longer PT8.3
Other:
- note added: "Populate these instead of IC12 if only 4 pots are needed"
- moved on the sheet: PT1, PT2, PT3, PT4, PT5, PT6, PT7, PT8

Commit message: update docs
Parts:
- IC10, IC11: value TEXAS_INSTRUMENTS_DAC8164IBPWG4TEXAS_INSTRUMENTS_DAC8164IBPWG4_0_1 -> DAC8164
Changed lines of the file:
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@@
 <attribute name="SPICEPREFIX" value="X"/>
 </part>
-<part name="IC11" library="ic_dac" deviceset="TEXAS_INSTRUMENTS_DAC8164IBPWG4" device="TEXAS_INSTRUMENTS_DAC8164IBPWG4_0_1"/>
-<part name="IC10" library="ic_dac" deviceset="TEXAS_INSTRUMENTS_DAC8164IBPWG4" device="TEXAS_INSTRUMENTS_DAC8164IBPWG4_0_1"/>
+<part name="IC11" library="ic_dac" deviceset="TEXAS_INSTRUMENTS_DAC8164IBPWG4" device="TEXAS_INSTRUMENTS_DAC8164IBPWG4_0_1" value="DAC8164"/>
+<part name="IC10" library="ic_dac" deviceset="TEXAS_INSTRUMENTS_DAC8164IBPWG4" device="TEXAS_INSTRUMENTS_DAC8164IBPWG4_0_1" value="DAC8164"/>
 <part name="SUPPLY34" library="supply" deviceset="GND" device="">
 <attribute name="SPICEPREFIX" value="G"/>
