File: hardware/teensy/xen_teensy_controls_template.brd (EAGLE design)
At the start: 69.9 x 110.5 mm, 89 parts, among them IC1 TL074D, IC5 TL074D

Commit message: update template
Parts:
- added 3.3VA, OFFSET: HEADER/MALE/01, connectors:HEADER/MALE/01
- moved GND9 1.27 mm to (1.27, 73.7)
- moved +12V 1.27 mm to (1.27, 68.6)
- moved -12V 1.27 mm to (1.27, 83.8)
- moved -5V 1.27 mm to (1.27, 71.1)
- moved 3.3V 1.27 mm to (1.27, 78.7)
- moved 5V 1.27 mm to (1.27, 81.3)
- renumbered CV10 to PT5, CV10_ to PT6, CV11 to PT3, CV11_ to PT4, CV12 to PT2, CV12_ to PT1, CV9 to PT8, CV9_ to PT7
