File: hardware/teensy/xen_teensy_controls_template.sch (EAGLE design)
At the start: 88 parts, among them IC1 TL074D, IC5 TL074D

Commit message: update template
Parts:
- added 3.3VA, OFFSET: HEADER/MALE/01, connectors:HEADER/MALE/01
- renumbered CV10 to PT5, CV10_ to PT6, CV11 to PT3, CV11_ to PT4, CV12 to PT2, CV12_ to PT1, CV9 to PT8, CV9_ to PT7
Changed lines of the file:
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@@
 <drawing>
 <settings>
-<setting alwaysvectorfont="no"/>
+<setting alwaysvectorfont="yes"/>
 <setting verticaltext="up"/>
 </settings>
@@
 <attribute name="SPICEPREFIX" value="X"/>
 </part>
-<part name="CV11_" library="connectors" deviceset="HEADER/MALE/01" device="">
-<attribute name="SPICEPREFIX" value="X"/>
-</part>
-<part name="CV11" library="connectors" deviceset="HEADER/MALE/01" device="">
-<attribute name="SPICEPREFIX" value="X"/>
-</part>
-<part name="CV10" library="connectors" deviceset="HEADER/MALE/01" device="">
-<attribute name="SPICEPREFIX" value="X"/>
-</part>
-<part name="CV10_" library="connectors" deviceset="HEADER/MALE/01" device="">
-<attribute name="SPICEPREFIX" value="X"/>
-</part>
-<part name="CV9" library="connectors" deviceset="HEADER/MALE/01" device="">
-<attribute name="SPICEPREFIX" value="X"/>
-</part>
-<part name="CV9_" library="connectors" deviceset="HEADER/MALE/01" device="">
-<attribute name="SPICEPREFIX" value="X"/>
-</part>
-<part name="CV12" library="connectors" deviceset="HEADER/MALE/01" device="">
-<attribute name="SPICEPREFIX" value="X"/>
-</part>
-<part name="CV12_" library="connectors" deviceset="HEADER/MALE/01" device="">
+<part name="PT4" library="connectors" deviceset="HEADER/MALE/01" device="">
+<attribute name="SPICEPREFIX" value="X"/>
+</part>
+<part name="PT3" library="connectors" deviceset="HEADER/MALE/01" device="">
+<attribute name="SPICEPREFIX" value="X"/>
+</part>
+<part name="PT5" library="connectors" deviceset="HEADER/MALE/01" device="">
+<attribute name="SPICEPREFIX" value="X"/>
+</part>
+<part name="PT6" library="connectors" deviceset="HEADER/MALE/01" device="">
+<attribute name="SPICEPREFIX" value="X"/>
+</part>
+<part name="PT8" library="connectors" deviceset="HEADER/MALE/01" device="">
+<attribute name="SPICEPREFIX" value="X"/>
+</part>
+<part name="PT7" library="connectors" deviceset="HEADER/MALE/01" device="">
+<attribute name="SPICEPREFIX" value="X"/>
+</part>
+<part name="PT2" library="connectors" deviceset="HEADER/MALE/01" device="">
+<attribute name="SPICEPREFIX" value="X"/>
+</part>
+<part name="PT1" library="connectors" deviceset="HEADER/MALE/01" device="">
 <attribute name="SPICEPREFIX" value="X"/>
 </part>
@@
 </part>
 <part name="10_IO_CS" library="connectors" deviceset="HEADER/MALE/01" device="">
+<attribute name="SPICEPREFIX" value="X"/>
+</part>
+<part name="3.3VA" library="connectors" deviceset="HEADER/MALE/01" device="">
+<attribute name="SPICEPREFIX" value="X"/>
+</part>
+<part name="OFFSET" library="connectors" deviceset="HEADER/MALE/01" device="">
 <attribute name="SPICEPREFIX" value="X"/>
 </part>
@@
 <attribute name="NAME" x="-11.176" y="-54.356" size="1.778" layer="96"/>
 </instance>
-<instance part="CV11_" gate="HEADER" x="2.54" y="-167.64" smashed="yes">
+<instance part="PT4" gate="HEADER" x="2.54" y="-167.64" smashed="yes">
 <attribute name="NAME" x="-11.176" y="-168.656" size="1.778" layer="96"/>
 </instance>
-<instance part="CV11" gate="HEADER" x="2.54" y="-165.1" smashed="yes">
+<instance part="PT3" gate="HEADER" x="2.54" y="-165.1" smashed="yes">
 <attribute name="NAME" x="-11.176" y="-166.116" size="1.778" layer="96"/>
 </instance>
-<instance part="CV10" gate="HEADER" x="2.54" y="-157.48" smashed="yes">
+<instance part="PT5" gate="HEADER" x="2.54" y="-157.48" smashed="yes">
 <attribute name="NAME" x="-11.176" y="-158.496" size="1.778" layer="96"/>
 </instance>
-<instance part="CV10_" gate="HEADER" x="2.54" y="-160.02" smashed="yes">
+<instance part="PT6" gate="HEADER" x="2.54" y="-160.02" smashed="yes">
 <attribute name="NAME" x="-11.176" y="-161.036" size="1.778" layer="96"/>
 </instance>
-<instance part="CV9" gate="HEADER" x="2.54" y="-149.86" smashed="yes">
+<instance part="PT8" gate="HEADER" x="2.54" y="-149.86" smashed="yes">
 <attribute name="NAME" x="-11.176" y="-150.876" size="1.778" layer="96"/>
 </instance>
-<instance part="CV9_" gate="HEADER" x="2.54" y="-152.4" smashed="yes">
+<instance part="PT7" gate="HEADER" x="2.54" y="-152.4" smashed="yes">
 <attribute name="NAME" x="-11.176" y="-153.416" size="1.778" layer="96"/>
 </instance>
-<instance part="CV12" gate="HEADER" x="2.54" y="-172.72" smashed="yes">
+<instance part="PT2" gate="HEADER" x="2.54" y="-172.72" smashed="yes">
 <attribute name="NAME" x="-11.176" y="-173.736" size="1.778" layer="96"/>
 </instance>
-<instance part="CV12_" gate="HEADER" x="2.54" y="-175.26" smashed="yes">
+<instance part="PT1" gate="HEADER" x="2.54" y="-175.26" smashed="yes">
 <attribute name="NAME" x="-11.176" y="-176.276" size="1.778" layer="96"/>
 </instance>
@@
 <attribute name="NAME" x="-11.176" y="26.924" size="1.778" layer="96"/>
 </instance>
+<instance part="3.3VA" gate="HEADER" x="2.54" y="88.9" smashed="yes">
+<attribute name="NAME" x="-11.176" y="87.884" size="1.778" layer="96"/>
+</instance>
+<instance part="OFFSET" gate="HEADER" x="2.54" y="-180.34" smashed="yes">
+<attribute name="NAME" x="-11.176" y="-181.356" size="1.778" layer="96"/>
+</instance>
 </instances>
