File: hardware/teensy/xen_teensy_motherboard_8cv4pt_mki.brd (EAGLE design)
At the start: 69.9 x 110.5 mm, 355 parts, among them IC1 TL074PW, IC10 DAC8164, IC11 DAC8164, IC12 CD4051CD4051_SO16, IC2 MCP23S17SO, IC3 MCP6004, IC4 MCP6004, IC5 TL074PW, IC6 TEENSY41-OUTER, IC7 R-78E5.0-0.5, IC8 LM4040-5V, IC9 3.3V, P1 HEADER/MALE/01NOBORDER, P10 HEADER/MALE/01NOBORDER, P11 HEADER/MALE/01NOBORDER, P12 HEADER/MALE/01NOBORDER, P13 HEADER/MALE/01NOBORDER, P14 HEADER/MALE/01NOBORDER, P15 HEADER/MALE/01NOBORDER, P16 HEADER/MALE/01NOBORDER, P17 HEADER/MALE/01NOBORDER, P18 HEADER/MALE/01NOBORDER, P19 HEADER/MALE/01NOBORDER, P2 HEADER/MALE/01NOBORDER, P21 HEADER/MALE/01NOBORDER, P22 HEADER/MALE/01NOBORDER, P23 HEADER/MALE/01NOBORDER, P24 HEADER/MALE/01NOBORDER, P25 HEADER/MALE/01NOBORDER, P26 HEADER/MALE/01NOBORDER, P27 HEADER/MALE/01NOBORDER, P28 HEADER/MALE/01NOBORDER, P29 HEADER/MALE/01NOBORDER, P3 HEADER/MALE/01NOBORDER, P30 HEADER/MALE/01NOBORDER, P31 HEADER/MALE/01NOBORDER, P32 HEADER/MALE/01NOBORDER, P33 HEADER/MALE/01NOBORDER, P34 HEADER/MALE/01NOBORDER, P35 HEADER/MALE/01NOBORDER, P36 HEADER/MALE/01NOBORDER, P37 HEADER/MALE/01NOBORDER, P38 HEADER/MALE/01NOBORDER, P39 HEADER/MALE/01NOBORDER, P4 HEADER/MALE/01NOBORDER, P40 HEADER/MALE/01NOBORDER, P41 HEADER/MALE/01NOBORDER, P42 HEADER/MALE/01NOBORDER, P44 HEADER/MALE/01NOBORDER, P45 HEADER/MALE/01NOBORDER, P46 HEADER/MALE/01NOBORDER, P47 HEADER/MALE/01NOBORDER, P49 HEADER/MALE/01NOBORDER, P5 HEADER/MALE/01NOBORDER, P50 HEADER/MALE/01NOBORDER, P6 HEADER/MALE/01NOBORDER, P7 HEADER/MALE/01NOBORDER, P8 HEADER/MALE/01NOBORDER, P9 HEADER/MALE/01NOBORDER, Q1 BF170, Q10 BF170, Q11 BF170, Q12 BF170, Q13 BF170, Q14 BF170, Q15 BF170, Q16 BF170, Q2 BF170, Q3 BF170, Q4 BF170, Q5 BF170, Q6 BF170, Q7 BF170, Q8 BF170, Q9 BF170

Commit message: updated hardware
Connections:
- net N$10: no longer R9.2
- net N$11: now also R9.2
- net N$15: no longer R16.2
- net N$17: now also R16.2
- net N$21: no longer R19.2
- net N$25: now also R19.2
- net N$3: no longer R1.2
- net N$33: no longer R39.2
- net N$4: now also R1.2
- net N$42: now also R39.2
- net N$44: no longer R42.2
- net N$47: now also R42.2
- net N$49: no longer R45.2
- net N$50: now also R45.2
- net N$6: no longer R4.2
- net N$7: now also R4.2
Routing:
- net N$6: track 19.0 -> 13.4 mm
- net N$3: track 35.9 -> 30.4 mm
- net N$21: track 60.5 -> 55.6 mm
- net N$33: track 46.2 -> 41.9 mm
- net N$49: track 63.7 -> 59.8 mm
- net N$44: track 41.9 -> 38.0 mm
- net N$10: track 17.0 -> 13.1 mm
- net N$15: track 38.3 -> 34.4 mm
