File: hardware/temp/xen_daisy_motherboard.brd (EAGLE design)
At the start: 69.9 x 105.4 mm, 210 parts, among them IC1 TL074D, IC2 MCP23S17SO, IC3 MCP6004, IC4 MCP6004, IC7 R-78E5.0-0.5, IC8 LM4040-5V, IC9 MCP6004, U1 ES_DAISY_SEED_REV4

Commit message: updated hardware
Parts:
- removed D1, D10, D11, D12, D13, D14, D15, D16, D2, D3, D4, D5, D6, D7, D8, D9: 3.3V, transistors:SOT23
- removed IC2: MCP23S17SO, ic_digital:SO28W
- removed IO1, IO10, IO11, IO12, IO13, IO14, IO15, IO16, IO2, IO3, IO4, IO5, IO6, IO7, IO8, IO9: HEADER/MALE/01, connectors:HEADER/MALE/01
- removed R56, R57, R58, R59, R60, R61, R72, R73, R74, R75, R76, R77, R78, R79, R80, R81, R82: 1k, resistors:R0603
Connections:
- removed net N$100: IO16.1, R73.2
- removed net N$101: IC2.18, R82.2
- removed net N$52: D1.3, IC2.21, R56.1
- removed net N$53: D2.3, IC2.22, R57.1
- removed net N$54: D3.3, IC2.23, R58.1
- removed net N$55: D4.3, IC2.24, R59.1
- removed net N$56: D5.3, IC2.25, R60.1
- removed net N$58: D6.3, IC2.26, R61.1
- removed net N$59: D7.3, IC2.27, R72.1
- removed net N$61: D8.3, IC2.28, R73.1
- removed net N$62: D9.3, IC2.1, R74.1
- removed net N$63: D10.3, IC2.2, R75.1
- removed net N$64: D11.3, IC2.3, R76.1
- removed net N$65: D12.3, IC2.4, R77.1
- removed net N$66: D13.3, IC2.5, R78.1
- removed net N$67: D14.3, IC2.6, R79.1
- removed net N$72: D15.3, IC2.7, R80.1
- removed net N$73: D16.3, IC2.8, R81.1
- removed net N$85: IO1.1, R74.2
- removed net N$86: IO2.1, R75.2
- removed net N$87: IO3.1, R76.2
- removed net N$88: IO4.1, R77.2
- removed net N$89: IO5.1, R78.2
- removed net N$90: IO6.1, R79.2
- removed net N$91: IO7.1, R80.2
- removed net N$92: IO8.1, R81.2
- removed net N$93: IO9.1, R56.2
- removed net N$94: IO10.1, R57.2
- removed net N$95: IO11.1, R58.2
- removed net N$96: IO12.1, R59.2
- removed net N$97: IO13.1, R60.2
- removed net N$98: IO14.1, R61.2
- removed net N$99: IO15.1, R72.2
- net 3.3V: no longer IC2.9, R82.1
- net PE: no longer D1.1, D10.1, D11.1, D12.1, D13.1, D14.1, D15.1, D16.1, D2.1, D3.1, D4.1, D5.1, D6.1, D7.1, D8.1, D9.1, IC2.10, IC2.15, IC2.16, IC2.17
- net SPI_IO_CS: no longer IC2.11
- net SPI_MISO: no longer IC2.14
- net SPI_MOSI: no longer IC2.13
- net SPI_SCK: no longer IC2.12
Routing:
- net PE: track 179.0 -> 108.9 mm, vias 14 -> 5
- net N$73: track 26.9 -> 0.00 mm
- net N$52: track 26.3 -> 0.00 mm
- net N$72: track 23.8 -> 0.00 mm
- net N$53: track 23.2 -> 0.00 mm
- net N$67: track 20.4 -> 0.00 mm
- net N$54: track 20.1 -> 0.00 mm
- net SPI_MISO: track 68.8 -> 49.7 mm
- net N$66: track 18.0 -> 0.00 mm
- net N$55: track 17.8 -> 0.00 mm
- net N$65: track 15.7 -> 0.00 mm
- net N$56: track 15.5 -> 0.00 mm
- net 3.3V: track 149.0 -> 134.0 mm, vias 5 -> 3
- net N$58: track 13.7 -> 0.00 mm
- net N$59: track 13.4 -> 0.00 mm
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