File: hardware/temp/xen_daisy_motherboard.sch (EAGLE design)
At the start: 205 parts, among them IC1 TL074D, IC2 MCP23S17SO, IC3 MCP6004, IC4 MCP6004, IC7 R-78E5.0-0.5, IC8 LM4040-5V, IC9 MCP6004, U1 ES_DAISY_SEED_REV4

Commit message: updated hardware
Parts:
- removed D1, D10, D11, D12, D13, D14, D15, D16, D2, D3, D4, D5, D6, D7, D8, D9: 3.3V, transistors:ZENER-DIODESOT23
- removed IC2: MCP23S17SO, ic_digital:MCP23S17SO
- removed IO1, IO10, IO11, IO12, IO13, IO14, IO15, IO16, IO2, IO3, IO4, IO5, IO6, IO7, IO8, IO9: HEADER/MALE/01, connectors:HEADER/MALE/01
- removed R56, R57, R58, R59, R60, R61, R72, R73, R74, R75, R76, R77, R78, R79, R80, R81, R82: 1k, resistors:RESISTOR
Connections:
- removed net N$100: IO16.3, R73.2
- removed net N$101: IC2.!RESET, R82.2
- removed net N$52: D1.C, IC2.GPA0, R56.1
- removed net N$53: D2.C, IC2.GPA1, R57.1
- removed net N$54: D3.C, IC2.GPA2, R58.1
- removed net N$55: D4.C, IC2.GPA3, R59.1
- removed net N$56: D5.C, IC2.GPA4, R60.1
- removed net N$58: D6.C, IC2.GPA5, R61.1
- removed net N$59: D7.C, IC2.GPA6, R72.1
- removed net N$61: D8.C, IC2.GPA7, R73.1
- removed net N$62: D9.C, IC2.GPB0, R74.1
- removed net N$63: D10.C, IC2.GPB1, R75.1
- removed net N$64: D11.C, IC2.GPB2, R76.1
- removed net N$65: D12.C, IC2.GPB3, R77.1
- removed net N$66: D13.C, IC2.GPB4, R78.1
- removed net N$67: D14.C, IC2.GPB5, R79.1
- removed net N$72: D15.C, IC2.GPB6, R80.1
- removed net N$73: D16.C, IC2.GPB7, R81.1
- removed net N$85: IO1.3, R74.2
- removed net N$86: IO2.3, R75.2
- removed net N$87: IO3.3, R76.2
- removed net N$88: IO4.3, R77.2
- removed net N$89: IO5.3, R78.2
- removed net N$90: IO6.3, R79.2
- removed net N$91: IO7.3, R80.2
- removed net N$92: IO8.3, R81.2
- removed net N$93: IO9.3, R56.2
- removed net N$94: IO10.3, R57.2
- removed net N$95: IO11.3, R58.2
- removed net N$96: IO12.3, R59.2
- removed net N$97: IO13.3, R60.2
- removed net N$98: IO14.3, R61.2
- removed net N$99: IO15.3, R72.2
- net 3.3V: no longer IC2.VDD, R82.1
- net PE: no longer D1.A, D10.A, D11.A, D12.A, D13.A, D14.A, D15.A, D16.A, D2.A, D3.A, D4.A, D5.A, D6.A, D7.A, D8.A, D9.A, IC2.A0, IC2.A1, IC2.A2, IC2.VSS
- net SPI_IO_CS: no longer IC2.!CS
- net SPI_MISO: no longer IC2.SO
- net SPI_MOSI: no longer IC2.SI
- net SPI_SCK: no longer IC2.SCK
Other:
- note removed: "OUTPUTS"
- moved on the sheet: -5V, AIN_L, AIN_R, AOUT_L, AOUT_R, C10, C11, C12, C13, C14, C16, C17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
